Commit message: changed person color to black for easy visualization

File: bwi_gazebo_entities/urdf/common.urdf.xacro (robot description, xacro)
@@ -10,4 +10,7 @@
     <color rgba="0.4 0.4 0.4 1" />
   </material>
+  <material name="black">
+    <color rgba="0.0 0.0 0.0 1" />
+  </material>
   <material name="red">
     <color rgba="1.0 0.0 0.0 1" />

File: bwi_gazebo_entities/urdf/person.urdf.xacro (robot description, xacro)
@@ -38,4 +38,7 @@
       </collision>
     </link>
+    <gazebo reference="base_link">
+      <material>Gazebo/Black</material>
+    </gazebo>
     <!-- depth perception lidar -->
     <joint name="lidar_joint" type="fixed">
@@ -72,7 +75,10 @@
           <cylinder length="0.9" radius="0.09" />
         </geometry>
-        <material name="dark_grey" />
-      </visual>
-    </link>
+        <material name="black" />
+      </visual>
+    </link>
+    <gazebo reference="left_leg_link">
+      <material>Gazebo/Black</material>
+    </gazebo>
     <xacro:default_surface name="left_leg" />
     <!-- right leg -->
@@ -95,7 +101,10 @@
           <cylinder length="0.9" radius="0.09" />
         </geometry>
-        <material name="dark_grey" />
-      </visual>
-    </link>
+        <material name="black" />
+      </visual>
+    </link>
+    <gazebo reference="right_leg_link">
+      <material>Gazebo/Black</material>
+    </gazebo>
     <xacro:default_surface name="right_leg" />
     <!-- head -->
@@ -117,7 +126,10 @@
           <sphere radius="0.15" />
         </geometry>
-        <material name="dark_grey" />
-      </visual>
-    </link>
+        <material name="black" />
+      </visual>
+    </link>
+    <gazebo reference="head_link">
+      <material>Gazebo/Black</material>
+    </gazebo>
     <!-- camera -->
     <joint name="camera_joint" type="fixed">
@@ -174,7 +186,10 @@
           <cylinder length="0.35" radius="0.07" />
         </geometry>
-        <material name="dark_grey" />
-      </visual>
-    </link>
+        <material name="black" />
+      </visual>
+    </link>
+    <gazebo reference="left_arm_link">
+      <material>Gazebo/Black</material>
+    </gazebo>
     <!-- left fore arm -->
     <joint name="left_forearm_joint" type="fixed">
@@ -196,7 +211,10 @@
           <cylinder length="0.35" radius="0.07" />
         </geometry>
-        <material name="dark_grey" />
-      </visual>
-    </link>
+        <material name="black" />
+      </visual>
+    </link>
+    <gazebo reference="left_forearm_link">
+      <material>Gazebo/Black</material>
+    </gazebo>
     <!-- right arm -->
     <joint name="right_arm_joint" type="fixed">
@@ -218,7 +236,10 @@
           <cylinder length="0.35" radius="0.07" />
         </geometry>
-        <material name="dark_grey" />
-      </visual>
-    </link>
+        <material name="black" />
+      </visual>
+    </link>
+    <gazebo reference="right_arm_link">
+      <material>Gazebo/Black</material>
+    </gazebo>
     <!-- right fore arm -->
     <joint name="right_forearm_joint" type="fixed">
@@ -240,7 +261,10 @@
           <cylinder length="0.35" radius="0.07" />
         </geometry>
-        <material name="dark_grey" />
-      </visual>
-    </link>
+        <material name="black" />
+      </visual>
+    </link>
+    <gazebo reference="right_forearm_link">
+      <material>Gazebo/Black</material>
+    </gazebo>
     <gazebo>
       <xacro:gazebo_person_drive />
